File: oskar_feet/hw/oskar_feet_rev1/oskar_feet_rev1.kicad_pcb (KiCad board)
At the start: 2 copper layers, 37 parts, among them J1 Conn_02x04_Odd_Even, J2 Conn_01x02_Male, J3 Conn_01x03_Male, J4 Conn_01x03_Male, J5 Conn_01x03_Male, J6 Conn_01x03_Male, K1 T92P11D22-12, U1 ATmega2560-16A, U2 MCP2515-xSO, U3 MCP2551-I-SN, Y1 Crystal_GND24, Y3 Crystal_GND24

Commit message: KICAD
Parts:
- removed kibuzzard-61FBB8CE: G***, kibuzzard-61FBB8CE
- added C12: TBD, Capacitor_THT:CP_Radial_D8.0mm_P2.50mm, F.Cu at (107.6, 90.6)
- added D2: LED, LED_SMD:LED_0603_1608Metric, F.Cu at (63.1, 117.7)
- added D3: LED, LED_SMD:LED_0603_1608Metric, F.Cu at (64.8, 117.7)
- added D4: LED, LED_SMD:LED_0603_1608Metric, F.Cu at (66.4, 117.7)
- added D5: LED, LED_SMD:LED_0603_1608Metric, F.Cu at (68.1, 117.7)
- added D6: LED, LED_SMD:LED_0603_1608Metric, F.Cu at (69.7, 117.7)
- added D7: LED, LED_SMD:LED_0603_1608Metric, F.Cu at (71.4, 117.8)
- added H1: MountingHole_Pad, MountingHole:MountingHole_4.3mm_M4_DIN965_Pad_TopBottom, F.Cu at (177.8, 152.4)
- added H2: MountingHole_Pad, MountingHole:MountingHole_4.3mm_M4_DIN965_Pad_TopBottom, F.Cu at (55.5, 66.0)
- added H3: MountingHole_Pad, MountingHole:MountingHole_4.3mm_M4_DIN965_Pad_TopBottom, F.Cu at (55.5, 151.9)
- added H4: MountingHole_Pad, MountingHole:MountingHole_4.3mm_M4_DIN965_Pad_TopBottom, F.Cu at (177.8, 66.0)
- added J10: Conn_01x04_Male, Connector_Molex:Molex_KK-254_AE-6410-04A_1x04_P2.54mm_Vertical, F.Cu at (81.9, 123.6)
- added J11: Conn_01x01_Male, Connector_PinHeader_2.54mm:PinHeader_1x01_P2.54mm_Vertical, F.Cu at (76.9, 132.9)
- added J12: Conn_01x01_Male, Connector_PinHeader_2.54mm:PinHeader_1x01_P2.54mm_Vertical, F.Cu at (74.4, 132.9)
- added J13: Conn_01x01_Male, Connector_PinHeader_2.54mm:PinHeader_1x01_P2.54mm_Vertical, F.Cu at (82.0, 132.9)
- added J14: Conn_01x01_Male, Connector_PinHeader_2.54mm:PinHeader_1x01_P2.54mm_Vertical, F.Cu at (71.9, 143.0)
- added J15: Conn_01x01_Male, Connector_PinHeader_2.54mm:PinHeader_1x01_P2.54mm_Vertical, F.Cu at (79.5, 132.9)
- added J16: Conn_01x01_Male, Connector_PinHeader_2.54mm:PinHeader_1x01_P2.54mm_Vertical, F.Cu at (71.9, 137.9)
- added J17: Conn_01x01_Male, Connector_PinHeader_2.54mm:PinHeader_1x01_P2.54mm_Vertical, F.Cu at (84.6, 132.9)
- added J18: Conn_01x01_Male, Connector_PinHeader_2.54mm:PinHeader_1x01_P2.54mm_Vertical, F.Cu at (71.9, 145.6)
- added J19: Conn_01x01_Male, Connector_PinHeader_2.54mm:PinHeader_1x01_P2.54mm_Vertical, F.Cu at (71.9, 140.5)
- added J20: Conn_01x01_Male, Connector_PinHeader_2.54mm:PinHeader_1x01_P2.54mm_Vertical, F.Cu at (71.9, 135.4)
- added J21: Conn_01x01_Male, Connector_PinHeader_2.54mm:PinHeader_1x01_P2.54mm_Vertical, F.Cu at (82.0, 148.1)
- added J22: Conn_01x01_Male, Connector_PinHeader_2.54mm:PinHeader_1x01_P2.54mm_Vertical, F.Cu at (87.1, 137.9)
- added J23: Conn_01x01_Male, Connector_PinHeader_2.54mm:PinHeader_1x01_P2.54mm_Vertical, F.Cu at (87.1, 145.6)
- added J24: Conn_01x01_Male, Connector_PinHeader_2.54mm:PinHeader_1x01_P2.54mm_Vertical, F.Cu at (87.1, 140.5)
- added J25: Conn_01x01_Male, Connector_PinHeader_2.54mm:PinHeader_1x01_P2.54mm_Vertical, F.Cu at (87.1, 143.0)
- added J26: Conn_01x01_Male, Connector_PinHeader_2.54mm:PinHeader_1x01_P2.54mm_Vertical, F.Cu at (74.4, 148.1)
- added J27: Conn_01x01_Male, Connector_PinHeader_2.54mm:PinHeader_1x01_P2.54mm_Vertical, F.Cu at (76.9, 148.1)
- added J28: Conn_01x01_Male, Connector_PinHeader_2.54mm:PinHeader_1x01_P2.54mm_Vertical, F.Cu at (87.1, 135.4)
- added J29: Conn_01x01_Male, Connector_PinHeader_2.54mm:PinHeader_1x01_P2.54mm_Vertical, F.Cu at (84.6, 148.1)
- added J30: Conn_01x01_Male, Connector_PinHeader_2.54mm:PinHeader_1x01_P2.54mm_Vertical, F.Cu at (79.5, 148.1)
- added J31: Conn_01x01_Male, Connector_PinHeader_2.54mm:PinHeader_1x01_P2.54mm_Vertical, F.Cu at (76.9, 135.4)
- added J32: Conn_01x01_Male, Connector_PinHeader_2.54mm:PinHeader_1x01_P2.54mm_Vertical, F.Cu at (82.0, 143.0)
- added J33: Conn_01x01_Male, Connector_PinHeader_2.54mm:PinHeader_1x01_P2.54mm_Vertical, F.Cu at (84.6, 137.9)
- added J34: Conn_01x01_Male, Connector_PinHeader_2.54mm:PinHeader_1x01_P2.54mm_Vertical, F.Cu at (76.9, 143.0)
- added J35: Conn_01x01_Male, Connector_PinHeader_2.54mm:PinHeader_1x01_P2.54mm_Vertical, F.Cu at (84.6, 140.5)
- added J36: Conn_01x01_Male, Connector_PinHeader_2.54mm:PinHeader_1x01_P2.54mm_Vertical, F.Cu at (84.6, 143.0)
- added J37: Conn_01x01_Male, Connector_PinHeader_2.54mm:PinHeader_1x01_P2.54mm_Vertical, F.Cu at (74.4, 137.9)
- added J38: Conn_01x01_Male, Connector_PinHeader_2.54mm:PinHeader_1x01_P2.54mm_Vertical, F.Cu at (76.9, 145.6)
- added J39: Conn_01x01_Male, Connector_PinHeader_2.54mm:PinHeader_1x01_P2.54mm_Vertical, F.Cu at (79.5, 137.9)
- added J40: Conn_01x01_Male, Connector_PinHeader_2.54mm:PinHeader_1x01_P2.54mm_Vertical, F.Cu at (74.4, 135.4)
- added J41: Conn_01x01_Male, Connector_PinHeader_2.54mm:PinHeader_1x01_P2.54mm_Vertical, F.Cu at (82.0, 135.4)
- added J42: Conn_01x01_Male, Connector_PinHeader_2.54mm:PinHeader_1x01_P2.54mm_Vertical, F.Cu at (74.4, 143.0)
- added J43: Conn_01x01_Male, Connector_PinHeader_2.54mm:PinHeader_1x01_P2.54mm_Vertical, F.Cu at (84.6, 135.4)
- added J44: Conn_01x01_Male, Connector_PinHeader_2.54mm:PinHeader_1x01_P2.54mm_Vertical, F.Cu at (79.5, 140.5)
- added J45: Conn_01x01_Male, Connector_PinHeader_2.54mm:PinHeader_1x01_P2.54mm_Vertical, F.Cu at (84.6, 145.6)
- added J46: Conn_01x01_Male, Connector_PinHeader_2.54mm:PinHeader_1x01_P2.54mm_Vertical, F.Cu at (82.0, 137.9)
- added J47: Conn_01x01_Male, Connector_PinHeader_2.54mm:PinHeader_1x01_P2.54mm_Vertical, F.Cu at (79.5, 143.0)
- added J48: Conn_01x01_Male, Connector_PinHeader_2.54mm:PinHeader_1x01_P2.54mm_Vertical, F.Cu at (74.4, 145.6)
- added J49: Conn_01x01_Male, Connector_PinHeader_2.54mm:PinHeader_1x01_P2.54mm_Vertical, F.Cu at (82.0, 145.6)
- added J50: Conn_01x01_Male, Connector_PinHeader_2.54mm:PinHeader_1x01_P2.54mm_Vertical, F.Cu at (82.0, 140.5)
- added J51: Conn_01x01_Male, Connector_PinHeader_2.54mm:PinHeader_1x01_P2.54mm_Vertical, F.Cu at (76.9, 140.5)
- added J52: Conn_01x01_Male, Connector_PinHeader_2.54mm:PinHeader_1x01_P2.54mm_Vertical, F.Cu at (74.4, 140.5)
- added J53: Conn_01x01_Male, Connector_PinHeader_2.54mm:PinHeader_1x01_P2.54mm_Vertical, F.Cu at (79.5, 145.6)
- added J54: Conn_01x01_Male, Connector_PinHeader_2.54mm:PinHeader_1x01_P2.54mm_Vertical, F.Cu at (79.5, 135.4)
- added J55: Conn_01x01_Male, Connector_PinHeader_2.54mm:PinHeader_1x01_P2.54mm_Vertical, F.Cu at (76.9, 137.9)
- added J56: Conn_01x01_Male, Connector_PinHeader_2.54mm:PinHeader_1x01_P2.54mm_Vertical, F.Cu at (91.5, 128.8)
- added J58: Conn_01x01_Male, Connector_PinHeader_2.54mm:PinHeader_1x01_P2.54mm_Vertical, F.Cu at (86.4, 123.7)
- added J59: Conn_01x01_Male, Connector_PinHeader_2.54mm:PinHeader_1x01_P2.54mm_Vertical, F.Cu at (89.0, 123.7)
- added J60: Conn_01x01_Male, Connector_PinHeader_2.54mm:PinHeader_1x01_P2.54mm_Vertical, F.Cu at (91.5, 123.7)
- added J61: Conn_01x01_Male, Connector_PinHeader_2.54mm:PinHeader_1x01_P2.54mm_Vertical, F.Cu at (94.1, 123.7)
- added J62: Conn_01x01_Male, Connector_PinHeader_2.54mm:PinHeader_1x01_P2.54mm_Vertical, F.Cu at (86.3, 126.2)
- added J63: Conn_01x01_Male, Connector_PinHeader_2.54mm:PinHeader_1x01_P2.54mm_Vertical, F.Cu at (88.9, 126.2)
- added J64: Conn_01x01_Male, Connector_PinHeader_2.54mm:PinHeader_1x01_P2.54mm_Vertical, F.Cu at (89.0, 128.8)
- added J65: Conn_01x01_Male, Connector_PinHeader_2.54mm:PinHeader_1x01_P2.54mm_Vertical, F.Cu at (86.4, 128.8)
- added J66: Conn_01x01_Male, Connector_PinHeader_2.54mm:PinHeader_1x01_P2.54mm_Vertical, F.Cu at (94.1, 126.2)
- added J67: Conn_01x01_Male, Connector_PinHeader_2.54mm:PinHeader_1x01_P2.54mm_Vertical, F.Cu at (91.4, 126.2)
- added J7: Conn_01x02_Female, Oskar:XT90, F.Cu at (163.5, 64.7)
- added J8: Conn_01x02_Male, Oskar:XT90, F.Cu at (116.6, 64.7)
- added J9: Conn_01x03_Male, Connector_Molex:Molex_KK-254_AE-6410-03A_1x03_P2.54mm_Vertical, F.Cu at (75.9, 74.0)
- added Q1: BC817, Package_TO_SOT_SMD:SOT-23, F.Cu at (93.7, 112.1)
- added R10: tbd, Resistor_SMD:R_0603_1608Metric, F.Cu at (68.1, 120.8)
- added R11: tbd, Resistor_SMD:R_0603_1608Metric, F.Cu at (69.7, 120.8)
- added R12: tbd, Resistor_SMD:R_0603_1608Metric, F.Cu at (71.4, 120.8)
- added R13: 10k, Resistor_SMD:R_0603_1608Metric, F.Cu at (82.0, 82.3)
- added R14: 10k, Resistor_SMD:R_0603_1608Metric, F.Cu at (82.0, 83.8)
- added R5: 330, Resistor_SMD:R_0603_1608Metric, F.Cu at (93.6, 114.9)
- added R6: 10k, Resistor_SMD:R_0603_1608Metric, F.Cu at (93.6, 116.6)
- added R7: tbd, Resistor_SMD:R_0603_1608Metric, F.Cu at (63.1, 120.8)
- added R8: tbd, Resistor_SMD:R_0603_1608Metric, F.Cu at (64.8, 120.8)
- added R9: tbd, Resistor_SMD:R_0603_1608Metric, F.Cu at (66.4, 120.8)
- added U4: MPRB4812LD-30W, Oskar:MPRB4812LD-30W, F.Cu at (108.3, 120.6)
- added kibuzzard-620D462F: G***, kibuzzard-620D462F, F.Cu at (116.3, 93.6)
- added kibuzzard-620D4636: G***, kibuzzard-620D4636, F.Cu at (163.6, 93.9)
- added kibuzzard-620D4649: G***, kibuzzard-620D4649, F.Cu at (170.5, 81.8)
- added kibuzzard-620D4649: G***, kibuzzard-620D4649, F.Cu at (109.6, 80.8)
- added kibuzzard-620F6F5F: G***, kibuzzard-620F6F5F, F.Cu at (78.3, 78.4)
- added kibuzzard-620F6F6C: G***, kibuzzard-620F6F6C, F.Cu at (78.3, 80.2)
- added kibuzzard-622DE651: G***, kibuzzard-622DE651, F.Cu at (85.2, 81.6)
- added kibuzzard-622E0128: G***, kibuzzard-622E0128, F.Cu at (64.8, 112.9)
- added kibuzzard-622E021D: G***, kibuzzard-622E021D, F.Cu at (66.4, 112.5)
- added kibuzzard-622E0245: G***, kibuzzard-622E0245, F.Cu at (63.1, 113.9)
- added kibuzzard-622E0709: G***, kibuzzard-622E0709, F.Cu at (69.7, 113.7)
- added kibuzzard-622E0714: G***, kibuzzard-622E0714, F.Cu at (68.1, 113.5)
- added kibuzzard-623B0250: G***, kibuzzard-623B0250, F.Cu at (78.1, 128.1)
- added kibuzzard-62568EE0: G***, kibuzzard-62568EE0, F.Cu at (74.0, 100.0)
- added kibuzzard-62568F06: G***, kibuzzard-62568F06, F.Cu at (71.4, 114.5)
- added kibuzzard-6256903B: G***, kibuzzard-6256903B, F.Cu at (94.7, 91.1)
- added kibuzzard-625E7F56: G***, kibuzzard-625E7F56, F.Cu at (69.1, 140.7)
- added kibuzzard-625E7F56: G***, kibuzzard-625E7F56, F.Cu at (79.4, 130.2)
- added kibuzzard-625E7F64: G***, kibuzzard-625E7F64, F.Cu at (89.8, 140.5)
- added kibuzzard-625E7F64: G***, kibuzzard-625E7F64, F.Cu at (79.1, 150.7)
- J1: value Conn_02x04_Odd_Even -> PROG
- moved C10 108.8 mm to (85.5, 95.4), turned to 90 degrees
- moved R4 95.2 mm to (87.0, 95.4), turned to 90 degrees
- moved C8 90.9 mm to (78.7, 83.0), turned to 90 degrees
- moved U2 88.3 mm to (78.5, 90.8), turned to -90 degrees
- moved Y1 86.9 mm to (75.8, 83.1), turned to 180 degrees
- moved C9 82.9 mm to (72.9, 83.2), turned to 90 degrees
- moved J3 61.7 mm to (97.6, 81.8)
- moved J4 61.7 mm to (87.9, 81.8)
- moved kibuzzard-61FBB893 61.7 mm to (105.5, 81.8)
- moved J5 61.7 mm to (87.9, 74.0)
- moved J6 61.7 mm to (97.6, 74.0)
- moved kibuzzard-61FBB827 61.7 mm to (105.5, 73.9)
- moved kibuzzard-61FBB8B4 61.7 mm to (85.1, 73.9)
- moved kibuzzard-61FBB948 61.7 mm to (100.2, 86.2)
- moved kibuzzard-61FBBAE0 61.7 mm to (90.4, 86.2)
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Connections:
- net Net-(C9-Pad1) renamed /OSC1
- net Net-(K1-Pad3) renamed +48V
- net Net-(U1-Pad33) renamed /XTAL2
- net Net-(U1-Pad34) renamed /XTAL1
- net Net-(U2-Pad7) renamed /OSC2
- K1 pad 1: unconnected-(K1-Pad1) -> Net-(K1-Pad1)
- K1 pad 2: unconnected-(K1-Pad2) -> +12V
- U1 pad 16: unconnected-(U1-Pad16) -> /WHEEL_ENGAGEMENT_LOWER
- U1 pad 17: unconnected-(U1-Pad17) -> /WHEEL_ENGAGEMENT_UPPER
- U1 pad 2: unconnected-(U1-Pad2) -> /CORNER_SENSOR_FL
- U1 pad 3: unconnected-(U1-Pad3) -> /CORNER_SENSOR_RL
- U1 pad 4: unconnected-(U1-Pad4) -> /CORNER_SENSOR_FR
- U1 pad 45: unconnected-(U1-Pad45) -> /LED1
- U1 pad 46: unconnected-(U1-Pad46) -> /LED2
- U1 pad 47: unconnected-(U1-Pad47) -> /LED3
- U1 pad 48: unconnected-(U1-Pad48) -> /LED4
- U1 pad 49: unconnected-(U1-Pad49) -> /LED5
- U1 pad 5: unconnected-(U1-Pad5) -> /CORNER_SENSOR_RR
- U1 pad 50: unconnected-(U1-Pad50) -> /LED6
- U1 pad 65: unconnected-(U1-Pad65) -> Net-(U1-Pad65)
- U1 pad 66: unconnected-(U1-Pad66) -> Net-(U1-Pad66)
- U1 pad 67: unconnected-(U1-Pad67) -> Net-(U1-Pad67)
- U1 pad 68: unconnected-(U1-Pad68) -> Net-(U1-Pad68)
- U1 pad 69: unconnected-(U1-Pad69) -> Net-(U1-Pad69)
- U1 pad 70: unconnected-(U1-Pad70) -> Net-(U1-Pad70)
- U1 pad 71: unconnected-(U1-Pad71) -> Net-(U1-Pad71)
- U1 pad 72: unconnected-(U1-Pad72) -> Net-(U1-Pad72)
- U1 pad 73: unconnected-(U1-Pad73) -> Net-(U1-Pad73)
- U1 pad 74: unconnected-(U1-Pad74) -> Net-(U1-Pad74)
- U1 pad 75: unconnected-(U1-Pad75) -> Net-(U1-Pad75)
- U1 pad 79: unconnected-(U1-Pad79) -> /MOTOR_PWR_EN
Routing:
- net +5V: track 31.0 -> 222.1 mm, vias 0 -> 4
- net +12V: track 0.00 -> 72.0 mm
- net Net-(K1-Pad1): track 0.00 -> 43.5 mm, vias 0 -> 1
- net +48V: track 16.0 -> 52.6 mm
- net /WHEEL_ENGAGEMENT_UPPER: track 0.00 -> 34.2 mm, vias 0 -> 2
- net /WHEEL_ENGAGEMENT_LOWER: track 0.00 -> 32.2 mm, vias 0 -> 3
- net Net-(U1-Pad73): track 0.00 -> 27.8 mm, vias 0 -> 1
- net Net-(U1-Pad74): track 0.00 -> 27.5 mm, vias 0 -> 1
- net /SCK: track 0.00 -> 24.7 mm, vias 0 -> 2
- net /CORNER_SENSOR_FL: track 12.6 -> 36.0 mm
- net /CORNER_SENSOR_RL: track 4.27 -> 26.1 mm
- net Net-(U1-Pad75): track 0.00 -> 21.8 mm
- net GND: track 30.0 -> 50.3 mm
- net /TXCAN: track 0.00 -> 20.0 mm, vias 0 -> 2
- net /RESET: track 2.54 -> 22.5 mm, vias 0 -> 1
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- added copper zone on B.Cu, net GND
- added copper zone on F.Cu, net GND
Other:
- board outline added: 133.2 x 96.8 mm
- board text added: "4x M4"
